File: latte-panda-carrier/GPIO.kicad_sch (KiCad schematic)
At the start: 0 parts

Commit message: 130.1
Add GPIO, I2C and UART.
Parts:
- added J10, J11, J14, J8: Conn_01x03_Pin, A_HDJ_Library:PinHeader_1x03_P2.54mm_Vertical, symbol Connector:Conn_01x03_Pin
- added J12, J13, J19, J20, J21, J7, J9: Conn_01x04, A_HDJ_Library:PinHeader_1x04_P2.54mm_Vertical, symbol Connector_Generic:Conn_01x04
- added U10, U11, U12, U17, U9: ULC0524P, A_HDJ_Library:Diodes_UDFN-10_1.0x2.5mm_P0.5mm, symbol Power_Protection:D3V3XA4B10LP
Connections:
- new net: U10.5, U10.6 (NC)
- new net: U12.5, U12.6 (NC)
- new net +3.3V: J13.1 (Pin_1), J13.2 (Pin_2), J13.3 (Pin_3), J13.4 (Pin_4), J14.1 (Pin_1), J14.2 (Pin_2), J14.3 (Pin_3), J21.1 (Pin_1), J21.2 (Pin_2), J21.3 (Pin_3), J21.4 (Pin_4)
- new net GND: J11.1 (Pin_1), J11.2 (Pin_2), J11.3 (Pin_3), J12.1 (Pin_1), J12.2 (Pin_2), J12.3 (Pin_3), J12.4 (Pin_4), J20.1 (Pin_1), J20.2 (Pin_2), J20.3 (Pin_3), J20.4 (Pin_4), U10.3 (VSS), U10.8 (VSS), U11.3 (VSS), U11.8 (VSS), U12.3 (VSS), U12.8 (VSS), U17.3 (VSS), U17.8 (VSS), U9.3 (VSS), U9.8 (VSS)
- new net GPP_D0: J19.4 (Pin_4), U17.1, U17.10 (NC)
- new net GPP_D1: J19.3 (Pin_3), U17.2, U17.9 (NC)
- new net GPP_D2: J19.2 (Pin_2), U17.4, U17.7 (NC)
- new net GPP_D3: J19.1 (Pin_1), U17.5, U17.6 (NC)
- new net I2C2_SCL: J9.4 (Pin_4), U11.1, U11.10 (NC)
- new net I2C2_SDA: J7.4 (Pin_4), U9.1, U9.10 (NC)
- new net I2C3_SCL: J9.3 (Pin_3), U11.2, U11.9 (NC)
- new net I2C3_SDA: J7.3 (Pin_3), U9.2, U9.9 (NC)
- new net I2C4_SCL: J9.2 (Pin_2), U11.4, U11.7 (NC)
- new net I2C4_SDA: J7.2 (Pin_2), U9.4, U9.7 (NC)
- new net I2C5_SCL: J9.1 (Pin_1), U11.5, U11.6 (NC)
- new net I2C5_SDA: J7.1 (Pin_1), U9.5, U9.6 (NC)
- new net SOC_UART0_RX: J8.1 (Pin_1), U10.1, U10.10 (NC)
- new net SOC_UART1_RX: J8.2 (Pin_2), U10.2, U10.9 (NC)
- new net SOC_UART2_RX: J8.3 (Pin_3), U10.4, U10.7 (NC)
- new net SOC_UART_0_TX: J10.1 (Pin_1), U12.1, U12.10 (NC)
- new net SOC_UART_1_TX: J10.2 (Pin_2), U12.2, U12.9 (NC)
- new net SOC_UART_2_TX: J10.3 (Pin_3), U12.4, U12.7 (NC)
Other:
- note added: "GPIO"
- note added: "I2C CONNECTORS"
- note added: "UART CONNECTORS"
