File: latte-panda-carrier/Ethernet.kicad_sch (KiCad schematic)
At the start: 0 parts

Commit message: 150
Add gigabit ethernet.
Parts:
- added C33, C34, C35, C36, C37, C39, C40, C41, C42, C43, C45, C48: 100nF/50V, A_HDJ_Library:C_0402_1005Metric, symbol Device:C
- added C38, C44: 10uF/50V, A_HDJ_Library:C_0402_1005Metric, symbol Device:C
- added C46, C47: 12pF/50V, A_HDJ_Library:C_0402_1005Metric, symbol Device:C
- added J6: RJ45_RB1-125B8G1A, A_HDJ_Library:RJ45_UDE_RB1-125B8G1A, symbol Connector:RJ45_RB1-125B8G1A
- added R20, R21: 10K/1%, A_HDJ_Library:R_0603_1608Metric, symbol Device:R
- added R22: 2.49K/1%, A_HDJ_Library:R_0603_1608Metric, symbol Device:R
- added R23: 1M/1%, symbol Device:R
- added R24, R25: 470R/1%, symbol Device:R
- added U6: RTL8111H-CG-RH, A_HDJ_Library:QFN-32-1EP_4x4mm_P0.4mm_EP2.65x2.65mm, symbol latte_hdj:RTL8111H-CG-RH
- added U7, U8: D3V3XA4B10LP, Package_DFN_QFN:Diodes_UDFN-10_1.0x2.5mm_P0.5mm, symbol Power_Protection:D3V3XA4B10LP
- added Y1: 25MHz, symbol Device:Crystal_GND24
Connections:
- new net: C47.1, R23.1, U6.28 (CKXTAL1), Y1.1
- new net: J6.L1, R25.1
- new net: C46.1, R23.2, U6.29 (CKXTAL2), Y1.3
- new net: C48.2, J6.R1 (CT)
- new net: J6.L3, R24.1
- new net: R20.2, U6.20 (ISOLATEB)
- new net: R21.2, U6.21 (LANWAKEB)
- new net: J6.L2, U6.25 (LED2)
- new net: J6.L4, U6.26 (LED1)
- new net: R22.1, U6.31 (RSET)
- new net +1V0: C33.2, C34.2, C35.2, C36.2, C40.2, C44.2, U6.22 (DVDD10), U6.24 (REGOUT), U6.3 (AVDD10), U6.30 (AVDD10), U6.8 (AVDD10)
- new net +3.3V: C37.2, C41.2, C45.2, R20.1, R21.1, R24.2, R25.2, U6.11 (AVDD33), U6.23 (VDDREG), U6.32 (AVDD33)
- new net GND: C33.1, C34.1, C35.1, C36.1, C37.1, C40.1, C41.1, C44.1, C45.1, C46.2, C47.2, C48.1, J6.R10 (GND), J6.SH, R22.2, U6.33 (GND), U7.3 (VSS), U7.8 (VSS), U8.3 (VSS), U8.8 (VSS), Y1.2, Y1.4
- new net GbE_PCIe_CLK+: U6.15 (REFCLK_P)
- new net GbE_PCIe_CLK-: U6.16 (REFCLK_N)
- new net GbE_PCIe_RX+: C43.2
- new net GbE_PCIe_RX-: C39.2
- new net GbE_PCIe_TX+: C42.2
- new net GbE_PCIe_TX-: C38.2
- new net HSI+: C42.1, U6.13 (HSIP)
- new net HSI-: C38.1, U6.14 (HSIN)
- new net HSO+: C43.1, U6.17 (HSOP)
- new net HSO-: C39.1, U6.18 (HSON)
- new net MDI0+: J6.R2 (TD1+), U6.1 (MDIP0), U8.1, U8.10 (NC)
- new net MDI0-: J6.R3 (TD1-), U6.2 (MDIN0), U8.2, U8.9 (NC)
- new net MDI1+: J6.R4 (TD2+), U6.4 (MDIP1), U8.4, U8.7 (NC)
- new net MDI1-: J6.R5 (TD2-), U6.5 (MDIN1), U8.5, U8.6 (NC)
- new net MDI2+: J6.R6 (TD3+), U6.6 (MDIP2), U7.2, U7.9 (NC)
- new net MDI2-: J6.R7 (TD3-), U6.7 (MDIN2), U7.1, U7.10 (NC)
- new net MDI3+: J6.R8 (TD4+), U6.9 (MDIP3), U7.5, U7.6 (NC)
- new net MDI3-: J6.R9 (TD4-), U6.10 (MDIN3), U7.4, U7.7 (NC)
- new net ~{PLT_RST}: U6.19 (PERSTB)
- no-connect marks 0 -> 2
