File: latte-panda-carrier/HDMI.kicad_sch (KiCad schematic)
At the start: 0 parts

Commit message: 170.2
Add HDMI.
Parts:
- added C17, C18, C19, C20, C21, C22, C23, C24, C25: 100nF/50V, A_HDJ_Library:C_0402_1005Metric, symbol Device:C_Small
- added D1, D2, D3: ESD5V0B03, A_HDJ_Library:D_0402_1005Metric, symbol Diode:ESD9B5.0ST5G
- added D4: 1N5819WS, PCM_JLCPCB:D_SOD-323, symbol PCM_JLCPCB-Diodes:Schottky,1N5819WS
- added F3: 6V/50mA, A_HDJ_Library:C_0603_1608Metric, symbol Device:Fuse
- added J3: HDMI_A, A_HDJ_Library:HDMI_A_Molex_208658-1001_Horizontal, symbol Connector:HDMI_A
- added Q1: 2N7002, A_HDJ_Library:SOT-23, symbol Transistor_FET:2N7002
- added Q2, Q3, Q4: 2SK3018, A_HDJ_Library:SOT-23, symbol Transistor_FET:2N7002
- added R10, R13, R14, R16, R17, R7, R8, R9: 470R/1%, A_HDJ_Library:R_0402_1005Metric, symbol Device:R
- added R11: 1K/1%, A_HDJ_Library:R_0402_1005Metric, symbol Device:R
- added R15, R18, R19, R3, R5: 2.2K/1%, A_HDJ_Library:R_0402_1005Metric, symbol Device:R
- added R4: 1M/1%, A_HDJ_Library:R_0402_1005Metric, symbol Device:R
- added R6: 21.5K/1%, A_HDJ_Library:R_0402_1005Metric, symbol Device:R
- added U1, U2: D3V3XA4B10LP, A_HDJ_Library:Diodes_UDFN-10_1.0x2.5mm_P0.5mm, symbol Power_Protection:D3V3XA4B10LP
Connections:
- new net: Q4.3 (D), R10.1, R13.1, R14.1, R16.1, R17.1, R7.1, R8.1, R9.1
- new net: Q1.2 (S), R11.1, R6.1
- new net: D2.2 (A2), J3.19 (HPD), R11.2
- new net: Q4.1 (G), R19.2
- new net: F3.2, J3.18 (+5V)
- new net +3.3V: Q1.1 (G), Q2.1 (G), Q3.1 (G), R3.1, R4.1, R5.1
- new net +5V: D4.2
- new net 5V_HDMI_VCC: C25.1, D4.1, F3.1, R15.1, R18.1
- new net DDC_SCL: D3.2 (A2), J3.15 (SCL), Q2.2 (S), R15.2
- new net DDC_SDA: D1.2 (A2), J3.16 (SDA), Q3.2 (S), R18.2
- new net DDI_B_DDC_SCL: Q2.3 (D), R5.2
- new net DDI_B_DDC_SDA: Q3.3 (D), R3.2
- new net DDI_B_HPD: Q1.3 (D), R4.2
- new net DDI_B_TX0+: C17.1
- new net DDI_B_TX0-: C18.1
- new net DDI_B_TX1+: C19.1
- new net DDI_B_TX1-: C20.1
- new net DDI_B_TX2+: C21.1
- new net DDI_B_TX2-: C22.1
- new net DDI_B_TX3+: C23.1
- new net DDI_B_TX3-: C24.1
- new net GND: C25.2, D1.1 (A1), D2.1 (A1), D3.1 (A1), J3.11 (CKS), J3.17 (GND), J3.2 (D2S), J3.5 (D1S), J3.8 (D0S), J3.SH, Q4.2 (S), R6.2, U1.3 (VSS), U1.8 (VSS), U2.3 (VSS), U2.8 (VSS)
- new net TMDS_CK+: C23.2, J3.10 (CK+), R8.2, U2.4, U2.7 (NC)
- new net TMDS_CK-: C24.2, J3.12 (CK-), R7.2, U2.5, U2.6 (NC)
- new net TMDS_D0+: C21.2, J3.7 (D0+), R10.2, U2.1, U2.10 (NC)
- new net TMDS_D0-: C22.2, J3.9 (D0-), R9.2, U2.2, U2.9 (NC)
- new net TMDS_D1+: C19.2, J3.4 (D1+), R14.2, U1.4, U1.7 (NC)
- new net TMDS_D1-: C20.2, J3.6 (D1-), R13.2, U1.5, U1.6 (NC)
- new net TMDS_D2+: C17.2, J3.1 (D2+), R17.2, U1.1, U1.10 (NC)
- new net TMDS_D2-: C18.2, J3.3 (D2-), R16.2, U1.2, U1.9 (NC)
- new net ~{PWR_LED}/~{PSON}: R19.1
- no-connect marks 0 -> 2
