File: latte-panda-carrier/M.2.kicad_sch (KiCad schematic)
At the start: 0 parts

Commit message: Add m.2
Schematics stuff should be done, now.
Parts:
- added C12, C51, C57, C59: 10uF/50V, A_HDJ_Library:C_0402_1005Metric, symbol Device:C_Small
- added C49, C50, C55, C56: 220nF/50V, A_HDJ_Library:C_0402_1005Metric, symbol Device:C_Small
- added C52, C53, C58, C60: 100nF/50V, A_HDJ_Library:C_0402_1005Metric, symbol Device:C_Small
- added D6: GREEN, A_HDJ_Library:LED_0603_1608Metric, symbol Device:LED
- added H7, H8: MountingHole_Pad, symbol Mechanical:MountingHole_Pad
- added J15: Bus_M.2_Socket_M, A_HDJ_Library:PCIe_M.2_Connectors_P=0.5mm_H=4.2mm_KeyM, symbol Connector:Bus_M.2_Socket_M
- added J16: Bus_M.2_Socket_E, A_HDJ_Library:PCIe_M.2_Connectors_P=0.5mm_H=4.2mm_KeyE, symbol Connector:Bus_M.2_Socket_E
- added R1, R12, R26, R29, R32: 0R/1%, A_HDJ_Library:R_0402_1005Metric, symbol Device:R
- added R34, R35: 10K/1%, A_HDJ_Library:R_0402_1005Metric, symbol Device:R
- added TP2: TestPoint, symbol Connector:TestPoint
Connections:
- new net: J16.56 (~{W_DISABLE1}), R34.1
- new net: J15.38 (DEVSLP), TP2.1
- new net: J15.69 (PEDET), R12.1
- new net: J16.50 (SUSCLK), R26.2
- new net: J16.54 (~{W_DISABLE2}), R35.1
- new net: D6.1 (K), J15.10 (DAS/~{DSS}/~{LED1})
- new net: J15.68 (SUSCLK), R29.1
- new net +3.3V: C12.1, C51.1, C52.1, C53.1, C57.1, C58.1, C59.1, C60.1, D6.2 (A), J15.12 (3.3V), J15.14 (3.3V), J15.16 (3.3V), J15.18 (3.3V), J15.2 (3.3V), J15.4 (3.3V), J15.70 (3.3V), J15.72 (3.3V), J15.74 (3.3V), J16.2 (3.3V), J16.4 (3.3V), J16.72 (3.3V), J16.74 (3.3V), R34.2, R35.2
- new net CON_PCIE_TX_1+: C49.2, C55.2, J15.49 (PETp0/SATA-A+), J16.35 (PETp0)
- new net CON_PCIE_TX_1-: C50.2, C56.2, J15.47 (PETn0/SATA-A-), J16.37 (PETn0)
- new net GND: C12.2, C51.2, C52.2, C53.2, C57.2, C58.2, C59.2, C60.2, H7.1, H8.1, J15.1 (GND), J15.15 (GND), J15.21 (GND), J15.27 (GND), J15.3 (GND), J15.33 (GND), J15.39 (GND), J15.45 (GND), J15.51 (GND), J15.57 (GND), J15.71 (GND), J15.73 (GND), J15.75 (GND), J15.9 (GND), J16.1 (GND), J16.18 (GND), J16.33 (GND), J16.39 (GND), J16.45 (GND), J16.51 (GND), J16.57 (GND), J16.63 (GND), J16.69 (GND), J16.7 (GND), J16.75 (GND), R1.2, R12.2, R32.2
- new net PCIE_RX_0+: J16.41 (PERp0)
- new net PCIE_RX_0-: J16.43 (PERn0)
- new net PCIE_RX_1+: J15.43 (PERp0/SATA-B-)
- new net PCIE_RX_1-: J15.41 (PERn0/SATA-B+)
- new net PCIE_TX_0+: C55.1
- new net PCIE_TX_0-: C56.1
- new net PCIE_TX_1+: C49.1
- new net PCIE_TX_1-: C50.1
- new net REFCLKE+: J16.47 (REFCLKp0)
- new net REFCLKE-: J16.49 (REFCLKn0)
- new net REFCLKM+: J15.55 (REFCLKp)
- new net REFCLKM-: J15.53 (REFCLKn)
- new net SUSCLK: R26.1, R29.2
- new net USB_2_P7+: J16.3 (USB_D+)
- new net USB_2_P7-: J16.5 (USB_D-)
- new net ~{CLK_REQE}: J16.53 (~{CLKREQ0}), R32.1
- new net ~{CLK_REQM}: J15.52 (~{CLKREQ}), R1.1
- new net ~{PLT_RST}: J15.50 (~{PERST}), J16.52 (~{PERST0})
- new net ~{WAKE}: J15.54 (~{PEWAKE}), J16.55 (~{PEWAKE0})
- no-connect marks 0 -> 50
